Commit message: robot_core.xacro changes

File: description/robot.urdf.xacro (robot description, xacro)
@@ -2,4 +2,4 @@
 <robot xmlns:xacro="http://www.ros.org/wiki/xacro"  name="robot">
     <!-- ****************** add all xacros here *******************************  -->
-    <link name="robot_core.xacro"></link>
+    <xacro:include filename="robot_core.xacro" />
 </robot>

File: description/robot_core.xacro (robot description, xacro)
@@ -1,5 +1,5 @@
 <?xml version="1.0"?>
-<robot xmlns:xacro="http://www.ros.org/wiki/xacro">
-<!-- ****************** ROBOT CONSTANTS *******************************  -->
+<robot name="daniel_bot" xmlns:xacro="http://ros.org/wiki/xacro">
+  <!-- ****************** ROBOT CONSTANTS *******************************  -->
   <!-- Definition of geometry parameters -->
   <!-- Gantry -->
@@ -44,5 +44,5 @@
     </inertial>
   </xacro:macro>
-<!-- ****************** COORDINATES ORIGIN ***************************  -->
+  <!-- ****************** COORDINATES ORIGIN ***************************  -->
   <!-- Define the center of the robot -->
   <link name="world" />
@@ -50,5 +50,5 @@
   <!-- The base origin is offset from the world origin. -->
   <joint name="gantry_joint" type="fixed">
-    <origin xyz="${gantry_length/2} ${gantry_length/2} ${gantry_length/2}" rpy="0 0 0" />
+    <origin xyz="0 0 0" rpy="0 0 0" />
     <parent link="world" />
     <child link="gantry_link" />
@@ -57,5 +57,5 @@
   <link name="gantry_link">
     <visual>
-      <origin xyz="0 0 -${gantry_length/2}" rpy="0 0 0" />
+      <origin xyz="0 0 ${-gantry_length/2}" rpy="0 0 0" />
       <geometry>
         <box size="${gantry_length} ${gantry_length} ${gantry_length}" />
@@ -77,5 +77,5 @@
   <link name="base_link">
     <visual>
-      <origin xyz="0 0 ${-gantry_length/2-base_length/2}" rpy="0 0 0" />
+      <origin xyz="0 0 ${-base_length/2}" rpy="0 0 0" />
       <geometry>
         <cylinder length="${base_length}" radius="${base_radius}" />
@@ -86,5 +86,5 @@
     </visual>
     <collision>
-      <origin xyz="0 0 ${-gantry_length/2-base_length/2}" rpy="0 0 0" />
+      <origin xyz="0 0 ${-base_length/2}" rpy="0 0 0" />
       <geometry>
         <cylinder length="${base_length}" radius="${base_radius}" />
@@ -94,7 +94,7 @@
   </link>
     <!-- Connect the GANTRY to the BASE -->
-  <joint name="$base_joint" type="revolute"> <!-- WAIST -->
+  <joint name="base_joint" type="revolute"> <!-- WAIST -->
     <parent link="gantry_link" />
-    <child link="$base_link" />
+    <child link="base_link" />
     <origin xyz="0 0 ${-gantry_length}" rpy="0 0 0" />
     <limit upper="${pi}" lower="-${pi}" effort="100" velocity="100" />
@@ -102,7 +102,7 @@
   </joint>
   <!-- *********************** BICEP ******************************  -->
-  <link name="$bicep_link">
+  <link name="bicep_link">
     <visual>
-      <origin xyz="0 0 0" rpy="0 0 0" />
+      <origin xyz="0 0 ${-bicep_length/2}" rpy="0 0 0" />
       <geometry>
         <box size="${bicep_width} ${bicep_height} ${bicep_length}" />
@@ -113,5 +113,5 @@
     </visual>
     <collision>
-      <origin xyz="0 0 0" rpy="0 0 0" />
+      <origin xyz="0 0 ${-bicep_length/2}" rpy="0 0 0" />
       <geometry>
         <box size="${bicep_width} ${bicep_height} ${bicep_length}" />
@@ -122,8 +122,8 @@
   </link>
   <!-- Connect the BICEP to the BASE -->
-  <joint name="$bicep_joint" type="revolute"> <!-- SHOULDER -->
+  <joint name="bicep_joint" type="revolute"> <!-- SHOULDER -->
     <parent link="base_link" />
-    <child link="$bicep_link" />
-    <origin xyz="0 0 ${-gantry_length-base_length}" rpy="0 0 0" />
+    <child link="bicep_link" />
+    <origin xyz="0 0 ${-base_length/2}" rpy="0 0 0" />
     <limit upper="${pi/2}" lower="-${pi/2}" effort="100" velocity="100" />
     <axis xyz="0 1 0" />

Commit message: create constants.xacro

File: description/robot.urdf.xacro (robot description, xacro)
@@ -3,3 +3,4 @@
     <!-- ****************** add all xacros here *******************************  -->
     <xacro:include filename="robot_core.xacro" />
+    <xacro:include filename="constants.xacro" />
 </robot>

File: description/robot_core.xacro (robot description, xacro)
@@ -1,47 +1,5 @@
 <?xml version="1.0"?>
 <robot name="daniel_bot" xmlns:xacro="http://ros.org/wiki/xacro">
-  <!-- ****************** ROBOT CONSTANTS *******************************  -->
-  <!-- Definition of geometry parameters -->
-  <!-- Gantry -->
-  <xacro:property name="gantry_length" value="0.5" /> <!-- El gantry es una caja de LxLxL -->
-  <xacro:property name="gantry_mass" value="1" />
-  <!-- Base -->
-  <xacro:property name="base_length" value="0.5" /> <!-- El eslabon BASE es un cilindro -->
-  <xacro:property name="base_radius" value="0.5" />
-  <xacro:property name="base_mass"   value="1" />
-  <!-- Bicep -->
-  <xacro:property name="bicep_length" value="5" /> <!-- El eslabon BICEP es una caja de WxHxL -->
-  <xacro:property name="bicep_width" value="0.5" />
-  <xacro:property name="bicep_height" value="0.5" />
-  <xacro:property name="bicep_mass" value="1" />
-  <!-- Forearm -->
-  <xacro:property name="forearm_length" value="0.5" /> <!-- El eslabon FOREARM es una caja de WxHxL -->
-  <xacro:property name="forearm_width" value="0.5" />
-  <xacro:property name="forearm_height" value="0.5" />
-  <xacro:property name="forearm_mass" value="1" />
-  <!-- Define intertial property macros  -->
-  <xacro:macro name="box_inertia" params="m w h d">
-    <inertial>
-      <origin xyz="0 0 0" rpy="${pi/2} 0 ${pi/2}" />
-      <mass value="${m}" />
-      <inertia ixx="${(m/12) * (h*h + d*d)}" ixy="0.0" ixz="0.0" iyy="${(m/12) * (w*w + d*d)}"
-        iyz="0.0" izz="${(m/12) * (w*w + h*h)}" />
-    </inertial>
-  </xacro:macro>
-  <xacro:macro name="cylinder_inertia" params="m r h">
-    <inertial>
-      <origin xyz="0 0 0" rpy="${pi/2} 0 0" />
-      <mass value="${m}" />
-      <inertia ixx="${(m/12) * (3*r*r + h*h)}" ixy="0" ixz="0" iyy="${(m/12) * (3*r*r + h*h)}"
-        iyz="0" izz="${(m/2) * (r*r)}" />
-    </inertial>
-  </xacro:macro>
-  <xacro:macro name="sphere_inertia" params="m r">
-    <inertial>
-      <mass value="${m}" />
-      <inertia ixx="${(2/5) * m * (r*r)}" ixy="0.0" ixz="0.0" iyy="${(2/5) * m * (r*r)}" iyz="0.0"
-        izz="${(2/5) * m * (r*r)}" />
-    </inertial>
-  </xacro:macro>
+ <xacro:include filename="constants.xacro" />
   <!-- ****************** COORDINATES ORIGIN ***************************  -->
   <!-- Define the center of the robot -->
