Commit message: Material is now in constants.xacro. Fixed framed is now world

File: description/constants.xacro (robot description, xacro)
@@ -7,21 +7,22 @@
     <xacro:property name="gantry_mass" value="1" />
     <!-- Base -->
-    <xacro:property name="base_length" value="0.5" /> <!-- El eslabon BASE es un cilindro -->
-    <xacro:property name="base_radius" value="0.5" />
+    <xacro:property name="base_length" value="0.25" /> <!-- El eslabon BASE es un cilindro -->
+    <xacro:property name="base_radius" value="0.05" />
     <xacro:property name="base_mass" value="1" />
     <!-- Bicep -->
-    <xacro:property name="bicep_length" value="5" /> <!-- El eslabon BICEP es una caja de WxHxL -->
-    <xacro:property name="bicep_width" value="0.5" />
-    <xacro:property name="bicep_height" value="0.5" />
+    <xacro:property name="bicep_length" value="0.45" /> <!-- El eslabon BICEP es una caja de WxHxL -->
+    <xacro:property name="bicep_width" value="0.05" />
+    <xacro:property name="bicep_height" value="0.05" />
     <xacro:property name="bicep_mass" value="1" />
     <!-- Forearm -->
-    <xacro:property name="forearm_length" value="0.5" /> <!-- El eslabon FOREARM es una caja de WxHxL -->
-    <xacro:property name="forearm_width" value="0.5" />
-    <xacro:property name="forearm_height" value="0.5" />
+    <xacro:property name="forearm_length" value="0.4" /> <!-- El eslabon FOREARM es una caja de WxHxL -->
+    <xacro:property name="forearm_width" value="0.05" />
+    <xacro:property name="forearm_height" value="0.05" />
     <xacro:property name="forearm_mass" value="1" />
-    <!-- Define intertial property macros  -->
-    <xacro:macro name="box_inertia" params="m w h d">
+    <!-- ****************** INERTIA *******************************  -->
+    <!-- Corregir la inercia. Hay que hacer steiner -->
+    <xacro:macro name="box_inertia" params="m w h d z">
         <inertial>
-            <origin xyz="0 0 0" rpy="${pi/2} 0 ${pi/2}" />
+            <origin xyz="0 0 ${z}" rpy="${pi/2} 0 ${pi/2}" />
             <mass value="${m}" />
             <inertia ixx="${(m/12) * (h*h + d*d)}" ixy="0.0" ixz="0.0" iyy="${(m/12) * (w*w + d*d)}"
@@ -45,3 +46,14 @@
         </inertial>
     </xacro:macro>
+    <!-- ****************** COLOR *******************************  -->
+    <xacro:property name="alpha" value="0.25" /> <!-- transparencia -->
+    <material name="red">
+        <color rgba="${255/255} ${0/255} ${0/255} ${alpha}" />
+    </material>
+    <material name="blue">
+        <color rgba="${0/255} ${0/255} ${255/255} ${alpha}" />
+    </material>
+    <material name="white">
+        <color rgba="${255/255} ${255/255} ${255/255} ${alpha}" />
+    </material>
 </robot>

File: description/robot.urdf.xacro (robot description, xacro)
@@ -3,4 +3,3 @@
     <!-- ****************** add all xacros here *******************************  -->
     <xacro:include filename="robot_core.xacro" />
-    <xacro:include filename="constants.xacro" />
 </robot>

File: description/robot_core.xacro (robot description, xacro)
@@ -8,5 +8,5 @@
   <!-- The base origin is offset from the world origin. -->
   <joint name="gantry_joint" type="fixed">
-    <origin xyz="0 0 0" rpy="0 0 0" />
+    <origin xyz="0 0 2" rpy="0 0 0" />
     <parent link="world" />
     <child link="gantry_link" />
@@ -15,14 +15,12 @@
   <link name="gantry_link">
     <visual>
-      <origin xyz="0 0 ${-gantry_length/2}" rpy="0 0 0" />
+      <origin xyz="0 0 ${gantry_length/2} " rpy="0 0 0" />
       <geometry>
         <box size="${gantry_length} ${gantry_length} ${gantry_length}" />
       </geometry>
-      <material name="Red">
-        <color rgba="${255/255} ${0/255} ${0/255} 0.5" />
-      </material>
+      <material name="red" />
     </visual>
     <collision>
-      <origin xyz="0 0 -${gantry_length/2}" rpy="0 0 0" />
+      <origin xyz="0 0 ${gantry_length/2}" rpy="0 0 0" />
       <geometry>
         <box size="${gantry_length} ${gantry_length} ${gantry_length}" />
@@ -30,19 +28,17 @@
     </collision>
     <xacro:box_inertia m="${gantry_mass}" w="${gantry_length}" d="${gantry_length}"
-      h="${gantry_length}" />
+      h="${gantry_length}" z="${gantry_length/2}"/>
   </link>
   <!-- ********************** BASE *********************************  -->
   <link name="base_link">
     <visual>
-      <origin xyz="0 0 ${-base_length/2}" rpy="0 0 0" />
+      <origin xyz="0 0 0" rpy="0 0 0" />
       <geometry>
         <cylinder length="${base_length}" radius="${base_radius}" />
       </geometry>
-      <material name="Red">
-        <color rgba="${255/255} ${0/255} ${0/255} 1.0" />
-      </material>
+      <material name="blue"/>
     </visual>
     <collision>
-      <origin xyz="0 0 ${-base_length/2}" rpy="0 0 0" />
+      <origin xyz="0 0 0" rpy="0 0 0" />
       <geometry>
         <cylinder length="${base_length}" radius="${base_radius}" />
@@ -55,5 +51,5 @@
     <parent link="gantry_link" />
     <child link="base_link" />
-    <origin xyz="0 0 ${-gantry_length}" rpy="0 0 0" />
+    <origin xyz="0 0 ${-base_length/2}" rpy="0 0 0" />
     <limit upper="${pi}" lower="-${pi}" effort="100" velocity="100" />
     <axis xyz="0 0 1" />
@@ -66,7 +62,5 @@
         <box size="${bicep_width} ${bicep_height} ${bicep_length}" />
       </geometry>
-      <material name="White">
-        <color rgba="${255/255} ${255/255} ${255/255} 1.0" />
-      </material>
+      <material name="white"/>
     </visual>
     <collision>
@@ -76,6 +70,6 @@
       </geometry>
     </collision>
-    <xacro:box_inertia m="${bicep_mass}" w="${bicep_width}" d="${bicep_height}"
-      h="${bicep_length}" /> <!-- Chequear bien cual es w d h !!!!!!!!!!!!-->
+    <xacro:box_inertia m="${bicep_mass}" w="${bicep_width}" d="${bicep_length}"
+      h="${bicep_height}" z="${-bicep_length/2}"/> <!-- Chequear bien cual es w d h !!!!!!!!!!!!-->
   </link>
   <!-- Connect the BICEP to the BASE -->
