Commit message: Forearm link and elbow joint added

File: description/robot_core.xacro (robot description, xacro)
@@ -1,5 +1,5 @@
 <?xml version="1.0"?>
 <robot name="daniel_bot" xmlns:xacro="http://ros.org/wiki/xacro">
- <xacro:include filename="constants.xacro" />
+  <xacro:include filename="constants.xacro" />
   <!-- ****************** COORDINATES ORIGIN ***************************  -->
   <!-- Define the center of the robot -->
@@ -28,5 +28,5 @@
     </collision>
     <xacro:box_inertia m="${gantry_mass}" w="${gantry_length}" d="${gantry_length}"
-      h="${gantry_length}" z="${gantry_length/2}"/>
+      h="${gantry_length}" z="${gantry_length/2}" />
   </link>
   <!-- ********************** BASE *********************************  -->
@@ -37,5 +37,5 @@
         <cylinder length="${base_length}" radius="${base_radius}" />
       </geometry>
-      <material name="blue"/>
+      <material name="blue" />
     </visual>
     <collision>
@@ -45,7 +45,7 @@
       </geometry>
     </collision>
-    <xacro:cylinder_inertia m="${base_mass}" r="${base_radius}" h="${base_length}"/>
+    <xacro:cylinder_inertia m="${base_mass}" r="${base_radius}" h="${base_length}" />
   </link>
-    <!-- Connect the GANTRY to the BASE -->
+  <!-- Connect the GANTRY to the BASE -->
   <joint name="base_joint" type="revolute"> <!-- WAIST -->
     <parent link="gantry_link" />
@@ -62,5 +62,5 @@
         <box size="${bicep_width} ${bicep_height} ${bicep_length}" />
       </geometry>
-      <material name="white"/>
+      <material name="white" />
     </visual>
     <collision>
@@ -71,5 +71,5 @@
     </collision>
     <xacro:box_inertia m="${bicep_mass}" w="${bicep_width}" d="${bicep_length}"
-      h="${bicep_height}" z="${-bicep_length/2}"/> <!-- Chequear bien cual es w d h !!!!!!!!!!!!-->
+      h="${bicep_height}" z="${-bicep_length/2}" /> <!-- Chequear bien cual es w d h !!!!!!!!!!!!-->
   </link>
   <!-- Connect the BICEP to the BASE -->
@@ -81,3 +81,29 @@
     <axis xyz="0 1 0" />
   </joint>
+ <!-- *********************** FOREARM ******************************  -->
+  <link name="forearm_link">
+    <visual>
+      <origin xyz="0 0 ${-forearm_length/2}" rpy="0 0 0" />
+      <geometry>
+        <box size="${forearm_width} ${forearm_height} ${forearm_length}" />
+      </geometry>
+      <material name="white" />
+    </visual>
+    <collision>
+      <origin xyz="0 0 ${-forearm_length/2}" rpy="0 0 0" />
+      <geometry>
+        <box size="${forearm_width} ${forearm_height} ${forearm_length}" />
+      </geometry>
+    </collision>
+    <xacro:box_inertia m="${forearm_mass}" w="${forearm_width}" d="${forearm_length}"
+      h="${forearm_height}" z="${-forearm_length/2}" /> <!-- Chequear bien cual es w d h !!!!!!!!!!!!-->
+  </link>
+  <!-- Connect the FOREARM to the BICEP -->
+  <joint name="forearm_joint" type="revolute"> <!-- ELBOW -->
+    <parent link="bicep_link" />
+    <child link="forearm_link" />
+    <origin xyz="0 0 ${-bicep_length}" rpy="0 0 0" />
+    <limit upper="${pi/2}" lower="-${pi/2}" effort="100" velocity="100" />
+    <axis xyz="0 1 0" />
+  </joint>
 </robot>

Commit message: modified:   description/robot_core.xacro

File: description/robot_core.xacro (robot description, xacro)
@@ -30,4 +30,7 @@
       h="${gantry_length}" z="${gantry_length/2}" />
   </link>
+     <gazebo reference="gantry_link">
+    <material>Gazebo/Yellow</material>
+  </gazebo>
   <!-- ********************** BASE *********************************  -->
   <link name="base_link">
@@ -55,4 +58,7 @@
     <axis xyz="0 0 1" />
   </joint>
+   <gazebo reference="base_link">
+    <material>Gazebo/Blue</material>
+  </gazebo>
   <!-- *********************** BICEP ******************************  -->
   <link name="bicep_link">
@@ -73,4 +79,7 @@
       h="${bicep_height}" z="${-bicep_length/2}" /> <!-- Chequear bien cual es w d h !!!!!!!!!!!!-->
   </link>
+  <gazebo reference="bicep_link">
+    <material>Gazebo/Yellow</material>
+  </gazebo>
   <!-- Connect the BICEP to the BASE -->
   <joint name="bicep_joint" type="revolute"> <!-- SHOULDER -->
@@ -99,4 +108,7 @@
       h="${forearm_height}" z="${-forearm_length/2}" /> <!-- Chequear bien cual es w d h   !!!!!!!!!!!!-->
   </link>
+  <gazebo reference="forearm_link">
+    <material>Gazebo/Blue</material>
+  </gazebo>
   <!-- Connect the FOREARM to the BICEP -->
   <joint name="forearm_joint" type="revolute"> <!-- ELBOW -->
